File: anura-split.kicad_pcb (KiCad board)
At the start: 2 copper layers, 118 x 96.4 mm, 48 parts, among them U1 Nice_Nano_V2

Commit message: 3d models added
removed dependencies for 3d models and instead integrated directly into
project
Parts:
- moved SW-BAT-1 16.9 mm to (439.5, 157.0)

Commit message: trace routing + silkscreen design
Parts:
- removed DS-L-1: Nice!View, anura:nice!view
- removed SW-BAT-1: SW_SPDT, anura:SW-TH_MSK12C02
- removed SW-RST-L1: SW_Push, anura:SW_PUSH_SPST
- added DS-1: Nice!View, anura:nice!view_rev2, F.Cu at (374.3, 159.7)
- added SW-BAT1: SW_SPDT, anura:SW-TH_MSK12C02, F.Cu at (435.5, 146.9)
- added SW-RST1: SW_Push, anura:SW_PUSH_SPST, F.Cu at (446.6, 163.1)
- BP-1: moved to B.Cu
- moved ? 14.6 mm to (376.5, 166.3)
- moved ? 12.7 mm to (295.1, 173.8)
- moved SW-2 12.7 mm to (354.1, 131.6)
- moved SW-3 12.7 mm to (354.1, 148.6)
- moved D-8 12.7 mm to (316.5, 114.9)
- moved SW-7 12.7 mm to (315.9, 104.1)
- moved SW-14 12.7 mm to (281.2, 147.1)
- moved D-1 12.7 mm to (354.1, 108.4)
- moved SW-13 12.7 mm to (278.5, 130.3)
- moved SW-17 12.7 mm to (349.0, 169.2)
- moved SW-4 12.7 mm to (336.1, 112.1)
- moved SW-10 12.7 mm to (297.1, 118.1)
- moved ? 12.7 mm to (363.9, 123.1)
- moved SW-5 12.7 mm to (336.1, 129.1)
- moved U1 12.7 mm to (374.3, 141.1)
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Routing:
- net COL-1: track 72.0 -> 176.3 mm
- net COL-2: track 72.0 -> 156.0 mm
- net COL-3: track 106.6 -> 186.5 mm, vias 5 -> 7
- net ROW-4: track 10.0 -> 69.8 mm, vias 1 -> 2
- net COL-4: track 81.0 -> 112.3 mm
- net COL-5: track 81.3 -> 99.8 mm
- net Net-(D-16-A): track 20.2 -> 29.7 mm
- net Net-(D-17-A): track 20.2 -> 29.7 mm
- net VBAT+: track 10.0 -> 17.8 mm, vias 1 -> 2
- net Net-(SW-BAT1-B): track 0.00 -> 4.97 mm, vias 0 -> 1
- net ENC-A: track 17.7 -> 21.5 mm
- net ROW-3: track 116.9 -> 113.9 mm
- net GND: track 32.6 -> 35.3 mm, vias 4 -> 5
- net +3V3: vias 1 -> 2
Other:
- board text added: "nice!view"

Commit message: routing + schematic changes
mcu nets reorganised to suit trace routing better, and more traces
routed
Parts:
- added ?: , , F.Cu at (362.4, 138.2)
- moved SW-2 5.98 mm to (349.8, 127.4)
- moved D-4 5.98 mm to (331.8, 101.8)
- moved ? 5.98 mm to (377.6, 162.1)
- moved ? 5.98 mm to (372.2, 162.1)
- moved D-1 5.98 mm to (349.8, 104.3)
- moved D-8 5.98 mm to (312.2, 110.8)
- moved D-9 5.98 mm to (313.1, 127.8)
- moved D-16 5.98 mm to (366.3, 167.4)
- moved D-17 5.98 mm to (346.3, 159.1)
- moved SW-16 5.98 mm to (363.3, 172.7)
- moved SW-7 5.98 mm to (311.6, 99.9)
- moved D-14 5.98 mm to (275.9, 136.8)
- moved CombChocEncoder1 5.98 mm to (324.8, 162.4)
- moved D-10 5.98 mm to (292.1, 107.9)
- moved D-18 5.98 mm to (335.8, 157.1)
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Connections:
- U1 pad 1: MISO -> unconnected-(U1-Pad1)
- U1 pad 10: ENC-A -> COL-1
- U1 pad 11: ENC-B -> ROW-4
- U1 pad 12: ROW-4 -> ENC-B
- U1 pad 13: COL-1 -> ENC-A
- U1 pad 14: COL-2 -> unconnected-(U1-16-Pad14)_1
- U1 pad 15: COL-3 -> unconnected-(U1-14-Pad15)_1
- U1 pad 16: COL-4 -> unconnected-(U1-15-Pad16)_1
- U1 pad 17: COL-5 -> unconnected-(U1-18-Pad17)
- U1 pad 18: unconnected-(U1-19-Pad18) -> ROW-3
- U1 pad 19: unconnected-(U1-20-Pad19)_1 -> ROW-2
- U1 pad 2: MOSI/SCL -> unconnected-(U1-0-Pad2)
- U1 pad 20: unconnected-(U1-21-Pad20)_1 -> ROW-1
- U1 pad 5: SCK/SDA -> unconnected-(U1-2-Pad5)
- U1 pad 6: CS -> COL-5
- U1 pad 7: ROW-1 -> COL-4
- U1 pad 8: ROW-2 -> COL-3
- U1 pad 9: ROW-3 -> COL-2
Routing:
- net COL-4: track 112.3 -> 158.7 mm, vias 5 -> 8
- net ROW-1: track 118.8 -> 153.8 mm, vias 1 -> 2
- net COL-3: track 186.5 -> 205.0 mm
- net COL-2: track 156.0 -> 171.6 mm
- net ROW-3: track 113.9 -> 128.7 mm
- net COL-1: track 176.3 -> 190.2 mm
- net COL-5: track 99.8 -> 113.6 mm
- net ROW-2: track 116.0 -> 129.1 mm
- net ROW-4: track 69.8 -> 81.3 mm
- net unconnected-(U1-0-Pad2): track 0.00 -> 10.0 mm, vias 0 -> 1
- net MOSI/SCL: track 10.0 -> 0.00 mm, vias 1 -> 0
- net unconnected-(U1-18-Pad17): track 0.00 -> 10.0 mm, vias 0 -> 1
- net MISO: track 10.0 -> 0.00 mm, vias 1 -> 0
- net unconnected-(U1-Pad1): track 0.00 -> 10.0 mm, vias 0 -> 1
- net CS: track 9.65 -> 0.00 mm, vias 1 -> 0
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